File: LVP_EcoDrive/LVP_EcoDrive.kicad_sch (KiCad schematic)
At the start: 54 parts, among them J1 Conn_02x05_Odd_Even, J10 Conn_01x02_Pin, J11 Conn_01x02_Pin, J12 Conn_01x02_Pin, J13 Conn_01x02_Pin, J2 Conn_02x05_Odd_Even, J3 Conn_02x05_Odd_Even, J4 Conn_02x05_Odd_Even, J5 Conn_02x05_Odd_Even, J6 Conn_02x20_Odd_Even, J7 Conn_01x02_Pin, J8 Conn_01x02_Pin, J9 Screw_Terminal_01x11, Q2 AO3400A, U1 SSIT3490EESA, U2 SSIT3490EESA, U3 SSIT3490EESA, U4 AMS1117-5.0, U5 LM311, U6 LM311, U7 LM311

Commit message: LVP_EcoDrive Done, Finalized
Parts:
- removed R19, R20: 330, Resistor_SMD:R_1206_3216Metric_Pad1.30x1.75mm_HandSolder, symbol Device:R
- added C10, C9: 100uF, Capacitor_SMD:CP_Elec_8x6.5, symbol Device:C_Polarized
- added C6: 10u, Capacitor_SMD:C_1206_3216Metric_Pad1.33x1.80mm_HandSolder, symbol Device:C
- added C7: 0.1u, Capacitor_SMD:C_1206_3216Metric_Pad1.33x1.80mm_HandSolder, symbol Device:C
- added C8: 47uF, Capacitor_SMD:CP_Elec_5x5.4, symbol Device:C_Polarized
- added D4: SMBJ5.0A_C83333, EasyEDA:SMB_L4.6-W3.6-LS5.3-RD, symbol EasyEDA:SMBJ5.0A_C83333
- added D5: SMBJ12A_C151251, EasyEDA:SMB_L4.6-W3.6-LS5.3-RD, symbol EasyEDA:SMBJ12A_C151251
- added J14: Conn_02x05_Odd_Even, Connector_IDC:IDC-Header_2x05_P2.54mm_Vertical, symbol Connector_Generic:Conn_02x05_Odd_Even
- added J15: Conn_01x05_Pin, Connector_PinHeader_1.27mm:PinHeader_1x05_P1.27mm_Vertical_SMD_Pin1Right, symbol Connector:Conn_01x05_Pin
- C1, C2, C3, C4, C5: footprint (none) -> Capacitor_SMD:C_1206_3216Metric_Pad1.33x1.80mm_HandSolder
- D1, D3: footprint LED_SMD:LED_1206_3216Metric_Pad1.42x1.75mm_HandSolder -> LED_SMD:LED_0603_1608Metric
- R1, R2, R3, R4, R5, R6: value 100 -> 220; footprint Resistor_SMD:R_1206_3216Metric_Pad1.30x1.75mm_HandSolder -> Resistor_SMD:R_0603_1608Metric_Pad0.98x0.95mm_HandSolder
- R16, R7: footprint Resistor_SMD:R_1206_3216Metric_Pad1.30x1.75mm_HandSolder -> Resistor_SMD:R_0603_1608Metric_Pad0.98x0.95mm_HandSolder
Connections:
- net +12V: now also C10.1, C6.1, C7.1, C9.1, D5.1 (K)
- net +5V: now also C8.1, D4.1, J14.9 (Pin_9)
- net ENC_R1: now also J6.8 (Pin_8), J15.1 (Pin_1); no longer J6.7 (Pin_7)
- net ENC_R2: now also J6.11 (Pin_11), J15.3 (Pin_3); no longer J6.9 (Pin_9)
- net ENC_R3: now also J6.12 (Pin_12), J15.4 (Pin_4); no longer J6.11 (Pin_11)
- net ENC_T1: now also J6.9 (Pin_9), J15.2 (Pin_2); no longer J6.8 (Pin_8)
- net EXP_CS0: now also J14.7 (Pin_7)
- net EXP_MISO: now also J14.5 (Pin_5)
- net EXP_MOSI: now also J14.3 (Pin_3)
- net EXP_SCLK: now also J14.1 (Pin_1)
- net FAN0: now also J6.24 (Pin_24); no longer J6.12 (Pin_12)
- net GND: now also C10.2, C6.2, C7.2, C8.2, C9.2, D4.2, D5.2 (A), J14.10 (Pin_10), J14.2 (Pin_2), J14.4 (Pin_4), J14.6 (Pin_6), J15.5 (Pin_5); no longer J6.24 (Pin_24)
- new net EXP_INT: J14.8 (Pin_8), J6.7 (Pin_7)
Other:
- moved on the sheet: C1, C2, C3, C4, C5, D1, D3, H1, H2, H3, H4, R16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

Commit message: Added : Fused Inputs for LVP
Parts:
- added F1, F2: Fuse_Small, Fuse:Fuse_2512_6332Metric, symbol Device:Fuse_Small
Connections:
- net +12V: now also F1.2; no longer J4.1 (Pin_1), J4.3 (Pin_3)
- net +5V: now also F2.2; no longer J4.5 (Pin_5)
- new net: F1.1, J4.1 (Pin_1), J4.3 (Pin_3)
- new net: F2.1, J4.5 (Pin_5)
Other:
- moved on the sheet: C8, D3, D4, R16
