File: ForgeX/LVP_E0/revA/LVP_EcoDrive.kicad_pcb (KiCad board)
At the start: 2 copper layers, 196 x 47.5 mm, 63 parts, among them J1 Conn_02x05_Odd_Even, J10 Conn_01x02_Pin, J11 Conn_01x02_Pin, J12 Conn_01x02_Pin, J13 Conn_01x02_Pin, J14 Conn_02x05_Odd_Even, J15 Conn_01x05_Pin, J2 Conn_02x05_Odd_Even, J3 Conn_02x05_Odd_Even, J4 Conn_02x05_Odd_Even, J5 Conn_02x05_Odd_Even, J6 Conn_02x20_Odd_Even, J7 Conn_01x02_Pin, J8 Conn_01x02_Pin, J9 Screw_Terminal_01x11, Q2 AO3400A, U1 SSIT3490EESA, U2 SSIT3490EESA, U3 SSIT3490EESA, U4 AMS1117-5.0, U5 LM311, U6 LM311, U7 LM311

Commit message: Major redesign & Reworks
* Star grounding scheme enforced across the whole ForgeX design....
* Viper26 based PSU designed
* Better signal integrity & decoupling on LVP and major reroute
* Laminated DC bus (Biplanar) , instead of (Coplanar) , for heavily reduced bus inductance & equivelant Electrolytics ESL
Parts:
- removed F1, F2: Fuse_Small, Fuse:Fuse_2512_6332Metric
- C3, C4, C5: footprint Capacitor_SMD:C_1206_3216Metric_Pad1.33x1.80mm_HandSolder -> Capacitor_SMD:C_0603_1608Metric_Pad1.08x0.95mm_HandSolder
- R17, R18, R21: footprint Resistor_SMD:R_1206_3216Metric_Pad1.30x1.75mm_HandSolder -> Resistor_SMD:R_0603_1608Metric_Pad0.98x0.95mm_HandSolder
- U4: value AMS1117-5.0 -> AMS1117-3.3; footprint Package_TO_SOT_SMD:SOT-223-3_TabPin2 -> Package_TO_SOT_SMD:SOT-89-3
- moved C8 57.1 mm to (231.8, 74.3), turned to -90 degrees
- moved C1 21.9 mm to (80.4, 74.2)
- moved C2 21.9 mm to (80.4, 76.6)
- moved U4 21.7 mm to (74.7, 75.7)
- moved R18 12.9 mm to (83.7, 91.4)
- moved R17 10.5 mm to (82.8, 93.9), turned to 180 degrees
- moved J15 10.3 mm to (234.1, 87.5)
- moved U7 9.74 mm to (100.4, 91.6)
- moved U5 9.74 mm to (87.5, 91.6)
- moved U6 9.74 mm to (93.8, 91.6)
- moved C7 8.68 mm to (104.4, 92.8), turned to 90 degrees
- moved R21 8.67 mm to (82.8, 95.5)
- moved C9 2.91 mm to (219.6, 64.8), turned to 90 degrees
- moved C5 2.31 mm to (240.5, 87.3)
- moved C3 1.98 mm to (240.4, 81.1)
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Connections:
- J4 pad 1: Net-(J4-Pin_1) -> +12V
- J4 pad 3: Net-(J4-Pin_1) -> /HVDC_Cnd
- J4 pad 4: GND -> /CBUS_Cnd
- J4 pad 5: Net-(J4-Pin_5) -> /BRAKE
- J4 pad 6: GND -> /PRECHARGE0
- J4 pad 7: /-12V -> /PRECHARGE1
- J4 pad 8: GND -> unconnected-(J4-Pin_8-Pad8)
- J5 pad 2: GND -> +12V
- J5 pad 3: /HVDC_Cnd -> GND
- J5 pad 4: /CBUS_Cnd -> GND
- J5 pad 5: /BRAKE -> +5V
- J5 pad 6: /PRECHARGE0 -> +5V
- J5 pad 7: /PRECHARGE1 -> GND
- J5 pad 8: unconnected-(J5-Pin_8-Pad8) -> GND
Routing:
- net GND: track 0.00 -> 42.8 mm, vias 377 -> 350
- net /PRECHARGE0: track 103.7 -> 65.1 mm
- net /CBUS_Cnd: track 113.6 -> 76.1 mm
- net /BRAKE: track 97.8 -> 61.5 mm
- net /PRECHARGE1: track 96.8 -> 61.7 mm
- net /HVDC_Cnd: track 114.3 -> 79.5 mm
- net /~{BKIN}: track 109.9 -> 86.9 mm, vias 3 -> 1
- net +5V: track 278.8 -> 300.2 mm, vias 19 -> 13
- net Net-(J4-Pin_5): track 13.9 -> 0.00 mm, vias 4 -> 0
- net +3.3V: track 42.1 -> 29.6 mm, vias 1 -> 2
- net +12V: track 268.6 -> 280.4 mm
- net /ENC_R3: track 84.9 -> 77.1 mm
- net Net-(J4-Pin_1): track 7.29 -> 0.00 mm
- net /HIN_{A}: track 93.8 -> 99.1 mm
- net /Csense_{A}: track 106.1 -> 100.9 mm, vias 4 -> 2
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- added copper zone on F.Cu, net +5V
- removed copper zone on F.Cu, net +12V
