File: ForgeX/LVP_E0/revA/LVP_EcoDrive.kicad_sch (KiCad schematic)
At the start: 63 parts, among them J1 Conn_02x05_Odd_Even, J10 Conn_01x02_Pin, J11 Conn_01x02_Pin, J12 Conn_01x02_Pin, J13 Conn_01x02_Pin, J14 Conn_02x05_Odd_Even, J15 Conn_01x05_Pin, J2 Conn_02x05_Odd_Even, J3 Conn_02x05_Odd_Even, J4 Conn_02x05_Odd_Even, J5 Conn_02x05_Odd_Even, J6 Conn_02x20_Odd_Even, J7 Conn_01x02_Pin, J8 Conn_01x02_Pin, J9 Screw_Terminal_01x11, Q2 AO3400A, U1 SSIT3490EESA, U2 SSIT3490EESA, U3 SSIT3490EESA, U4 AMS1117-5.0, U5 LM311, U6 LM311, U7 LM311

Commit message: Major redesign & Reworks
* Star grounding scheme enforced across the whole ForgeX design....
* Viper26 based PSU designed
* Better signal integrity & decoupling on LVP and major reroute
* Laminated DC bus (Biplanar) , instead of (Coplanar) , for heavily reduced bus inductance & equivelant Electrolytics ESL
Parts:
- removed F1, F2: Fuse_Small, Fuse:Fuse_2512_6332Metric, symbol Device:Fuse_Small
- removed U4: AMS1117-5.0, Package_TO_SOT_SMD:SOT-223-3_TabPin2, symbol Regulator_Linear:AMS1117-5.0
- added U4: AMS1117-3.3, Package_TO_SOT_SMD:SOT-89-3, symbol Regulator_Linear:AMS1117-3.3
- C3, C4, C5: footprint Capacitor_SMD:C_1206_3216Metric_Pad1.33x1.80mm_HandSolder -> Capacitor_SMD:C_0603_1608Metric_Pad1.08x0.95mm_HandSolder
- R17, R18, R21: footprint Resistor_SMD:R_1206_3216Metric_Pad1.30x1.75mm_HandSolder -> Resistor_SMD:R_0603_1608Metric_Pad0.98x0.95mm_HandSolder
- renumbered J5 to J4, J4 to J5
Connections:
- net -12V is gone; now on net GND: J5.7 (Pin_7)
- net +12V: now also J5.1 (Pin_1), J5.2 (Pin_2)
- net +3.3V: now also U4.2 (VO)
- net +5V: now also J5.5 (Pin_5), J5.6 (Pin_6), U4.3 (VI)
- net GND: now also J5.3 (Pin_3), U4.1 (GND); no longer J5.2 (Pin_2), J5.6 (Pin_6)
