File: ForgeX/LVP_G0S4/revA/LVP_G0S4.kicad_sch (KiCad schematic)
At the start: 64 parts, among them J1 Conn_02x05_Odd_Even, J10 Conn_01x02_Pin, J11 Conn_01x02_Pin, J12 Conn_01x02_Pin, J13 Conn_01x02_Pin, J14 Conn_02x05_Odd_Even, J15 Conn_01x05_Pin, J16 Conn_01x04, J17 Conn_01x04, J2 Conn_02x05_Odd_Even, J3 Conn_02x05_Odd_Even, J4 Conn_02x05_Odd_Even, J6 Conn_02x20_Odd_Even, J7 Conn_01x02_Pin, J8 Conn_01x02_Pin, J9 Screw_Terminal_01x11, Q2 AO3400A, U1 SSIT3490EESA, U2 SSIT3490EESA, U3 SSIT3490EESA, U4 AMS1117-3.3, U5 LM311, U6 LM311, U7 LM311

Commit message: BlackDev Fini & HBM mod
Finalized blackDev, HBM with (RC) ground coupling, LVP swapping RS422 to RS485 and processing card interface modifications
Parts:
- removed C5: 0.1u, Capacitor_SMD:C_0603_1608Metric_Pad1.08x0.95mm_HandSolder, symbol Device:C
- removed J15: Conn_01x05_Pin, Connector_PinHeader_1.27mm:PinHeader_1x05_P1.27mm_Vertical_SMD_Pin1Right, symbol Connector:Conn_01x05_Pin
- removed J9: Screw_Terminal_01x11, Connector_JST:JST_XH_B11B-XH-A_1x11_P2.50mm_Vertical, symbol Connector:Screw_Terminal_01x11
- removed U1, U2, U3: SSIT3490EESA, EasyEDA:SOIC-8_L5.0-W4.0-P1.27-LS6.0-BL, symbol EasyEDA:SSIT3490EESA
- added C11: 0.1u, Capacitor_SMD:C_0603_1608Metric_Pad1.08x0.95mm_HandSolder, symbol Device:C
- added D7, D8, D9: SD103AWS_C5345966, EasyEDA:SOD-323_L1.7-W1.3-LS2.5-RD, symbol EasyEDA:SD103AWS_C5345966
- added J5: Conn_01x04_Pin, Connector_PinHeader_1.27mm:PinHeader_1x04_P1.27mm_Vertical_SMD_Pin1Right, symbol Connector:Conn_01x04_Pin
- added J9: Screw_Terminal_01x09, Connector_JST:JST_XH_B9B-XH-A_1x09_P2.50mm_Vertical, symbol Connector:Screw_Terminal_01x09
- added JP1: SolderJumper_3_Bridged12, Jumper:SolderJumper-3_P1.3mm_Bridged12_RoundedPad1.0x1.5mm, symbol Jumper:SolderJumper_3_Bridged12
- added JP2: SolderJumper_2_Open, Jumper:SolderJumper-2_P1.3mm_Open_TrianglePad1.0x1.5mm, symbol Jumper:SolderJumper_2_Open
- added R19: 10k, Resistor_SMD:R_0603_1608Metric_Pad0.98x0.95mm_HandSolder, symbol Device:R
- added R20, R22, R23: 220, Resistor_SMD:R_0603_1608Metric_Pad0.98x0.95mm_HandSolder, symbol Device:R
- added U1, U2, U3: SP485EEN-TD, EasyEDA:SOIC-8_L4.9-W3.9-P1.27-LS6.0-BL, symbol EasyEDA:SP485EEN-TD
- J6: footprint Connector_IDC:IDC-Header_2x20_P2.54mm_Vertical -> Connector_PinSocket_2.54mm:PinSocket_2x20_P2.54mm_Vertical
Connections:
- net ENC_T1 is gone; now on net ENC_R1: J6.16 (Pin_16)
- net +12V: now also J6.26 (Pin_26); no longer J6.25 (Pin_25)
- net +3.3V: now also D7.1 (K), D8.1 (K), D9.1 (K)
- net +5V: now also J6.28 (Pin_28), C11.1, J9.7 (Pin_7), R19.1, U1.8 (VCC), U2.8 (VCC), U3.8 (VCC); no longer J6.27 (Pin_27)
- net Csense_{A}: now also J6.29 (Pin_29); no longer J6.30 (Pin_30)
- net Csense_{B}: now also J6.32 (Pin_32); no longer J6.31 (Pin_31)
- net Csense_{C}: now also J6.31 (Pin_31); no longer J6.32 (Pin_32)
- net ENC_R1: now also D9.2 (A), R23.2; no longer J6.15 (Pin_15)
- net ENC_R1+: now also J9.2 (Pin_2), U1.6 (A)
- net ENC_R1-: now also J9.1 (Pin_1), U1.7 (B)
- net ENC_R2: now also J6.14 (Pin_14), D7.2 (A), R20.2; no longer J6.13 (Pin_13)
- net ENC_R2+: now also J9.4 (Pin_4), U2.6 (A)
- net ENC_R2-: now also J9.3 (Pin_3), U2.7 (B)
- net ENC_R3: now also J6.11 (Pin_11), D8.2 (A), R22.2; no longer J6.12 (Pin_12)
- net ENC_R3+: now also J9.6 (Pin_6), U3.6 (A)
- net ENC_R3-: now also J9.5 (Pin_5), U3.7 (B)
- net EXP_MISO: now also J6.6 (Pin_6); no longer J6.5 (Pin_5)
- net EXP_MOSI: now also J6.4 (Pin_4); no longer J6.3 (Pin_3)
- net EXP_RX: now also J6.12 (Pin_12); no longer J6.11 (Pin_11)
- net EXP_SCLK: now also J6.2 (Pin_2); no longer J6.1 (Pin_1)
- net EXP_TX: now also J6.10 (Pin_10); no longer J6.9 (Pin_9)
- net Earth: now also J9.9 (Pin_9)
- net FAN0: now also J6.23 (Pin_23); no longer J6.24 (Pin_24)
- net GND: now also J6.1 (Pin_1), J6.13 (Pin_13), J6.25 (Pin_25), J6.27 (Pin_27), J6.3 (Pin_3), J6.39 (Pin_39), J6.5 (Pin_5), J6.9 (Pin_9), C11.2, J5.4 (Pin_4), J9.8 (Pin_8), JP2.2 (B), U1.5 (GND), U2.2 (~{RE}), U2.3 (DE), U2.5 (GND), U3.2 (~{RE}), U3.3 (DE), U3.5 (GND); no longer J6.10 (Pin_10), J6.14 (Pin_14), J6.2 (Pin_2), J6.26 (Pin_26), J6.28 (Pin_28), J6.4 (Pin_4), J6.40 (Pin_40), J6.6 (Pin_6)
- net HVDC_Cnd: now also J6.34 (Pin_34); no longer J6.33 (Pin_33)
- net Phase_Cnd_{A}: now also J6.33 (Pin_33); no longer J6.34 (Pin_34)
- net Phase_Cnd_{B}: now also J6.35 (Pin_35); no longer J6.36 (Pin_36)
- net Phase_Cnd_{C}: now also J6.36 (Pin_36); no longer J6.35 (Pin_35)
- net TEMP1: now also J6.38 (Pin_38); no longer J6.37 (Pin_37)
- net TEMP2: now also J6.37 (Pin_37); no longer J6.38 (Pin_38)
- net TEMP3: now also J6.40 (Pin_40); no longer J6.39 (Pin_39)
- net ~{BKIN}: now also J6.24 (Pin_24); no longer J6.23 (Pin_23)
- net at J6.17 (Pin_17): now also R2.2; no longer R1.1
- net at J6.18 (Pin_18): now also R1.1; no longer R2.2
- net at J6.19 (Pin_19): now also R5.2; no longer R3.1
- net at J6.20 (Pin_20): now also R3.1; no longer R5.2
- net at J6.21 (Pin_21): now also R6.2; no longer R4.1
- net at J6.22 (Pin_22): now also R4.1; no longer R6.2
- net EXP_INT renamed EXP_CS1
- new net: JP2.1 (A), R19.2, U1.2 (~{RE}), U1.3 (DE)
- new net: JP1.3 (B), U1.1 (RO)
- new net: JP1.1 (A), U1.4 (DI)
- new net ENC_R1P: J5.1 (Pin_1), JP1.2 (C), R23.1
- new net ENC_R2P: J5.2 (Pin_2), R20.1, U2.1 (RO)
- new net ENC_R3P: J5.3 (Pin_3), R22.1, U3.1 (RO)
- new net EXP_CS2: J6.15 (Pin_15)
- no-connect marks 28 -> 24
Other:
- moved on the sheet: C3, C4, C7, R12, R14, R15, R17, R18, R21, U5, U6
